File: board/foxie_clock_nano.kicad_pcb (KiCad board)
At the start: 2 copper layers, 166 x 55.5 mm, 133 parts, among them SW1 BTN_Hour, SW2 BTN_Minute, SW3 BTN_Color, SW4 BTN_Brightness, U1 SN74AHCT125N, U2 Artemis-Nano

Commit message: Minor wording change on PCB
Parts:
- moved C1 195.0 mm to (-42.9, -51.4)
- moved C2 195.0 mm to (-6.00, -51.4)
- moved C3 195.0 mm to (26.9, -51.4)
- moved C4 195.0 mm to (63.9, -51.4)
- moved D1 195.0 mm to (-62.6, -44.1)
- moved D10 195.0 mm to (-49.6, -29.1)
- moved D100 195.0 mm to (58.4, -10.6)
- moved D101 195.0 mm to (77.4, -44.1)
- moved D102 195.0 mm to (90.4, -44.1)
- moved D103 195.0 mm to (71.4, -40.6)
- moved D104 195.0 mm to (84.4, -40.6)
- moved D105 195.0 mm to (77.4, -36.6)
- moved D106 195.0 mm to (90.4, -36.6)
- moved D107 195.0 mm to (71.4, -33.1)
- moved D108 195.0 mm to (84.4, -33.1)
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Other:
- board outline removed
- board text added: "Thanks to JLC, www.kicad-pcb.org, www.arduino.cc, www.sparkfun.com, and makers like you! Also, thanks to Mel Brooks for Spaceballs."
- board text added: "v1.41, by Will Fox foxieproducts.com"
- board text removed: "Thanks to www.kicad-pcb.org, www.arduino.cc, www.sparkfun.com, and makers like you! Also, thanks to Mel Brooks for Spaceballs."
- board text removed: "v1.4, by Alex Fox alex@neg.plus"
